Commit message: first_commit_rma

File: resources/robots/bolt10/urdf/bolt10.urdf (robot description, URDF)
Before this commit: robot bolt10_urdf, 11 links, 10 joints
Joints:
- joint L_AnklePitch_Joint: limit lower=-1.50 upper=1.50 effort=3.5 velocity=50 -> lower=-1.0 upper=1.50 effort=3.5 velocity=50
- joint R_AnklePitch_Joint: limit lower=-1.50 upper=1.50 effort=3.5 velocity=50 -> lower=-1.00 upper=1.50 effort=3.5 velocity=50
